Commit message: update urdf

File: src/allegro_hand_description/allegro_hand_v4_right.urdf (robot description, URDF)
Before this commit: robot allegro_hand, 21 links, 20 joints
Links:
- removed link base_link
- added link palm_link, mass 4.1685782e-01; collision mesh filename=package://allegro_hand_description/meshes_v4/40_10_link_g_r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 scale=0.001 0.001 0.001; visual mesh filename=package://allegro_hand_description/meshes_v4/40_10_link_g_r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 scale=0.001 0.001 0.001
Joints:
- joint jif1: parent base_link -> palm_link
- joint jmf1: parent base_link -> palm_link
- joint jpf1: parent base_link -> palm_link
- joint jth1: parent base_link -> palm_link
